Commit message: update: add coustom hardware interface for esp serial communication with moveit

File: src/my_robot_description/urdf/volvo_arm.ros2_control.xacro (robot description, xacro)
@@ -1,45 +1,45 @@
 <?xml version="1.0"?>
 <robot xmlns:xacro="http://www.ros.org/wiki/xacro">
-    <ros2_control name="Volvo_Arm" type="system">
-            <hardware>
-                <!-- By default, set up controllers for simulation. This won't work on real hardware -->
-                <plugin>mock_components/GenericSystem</plugin>
-            </hardware>
-            <joint name="Joint_1">
-                <command_interface name="position"/>
-                <state_interface name="position">
-                  <param name="initial_value">0.0</param>
-                </state_interface>
-            </joint>
-            <joint name="Joint_2">
-                <command_interface name="position"/>
-                <state_interface name="position">
-                  <param name="initial_value">0.0</param>
-                </state_interface>
-            </joint>
-            <joint name="Joint_3">
-                <command_interface name="position"/>
-                <state_interface name="position">
-                  <param name="initial_value">0.0</param>
-                </state_interface>
-            </joint>
-            <joint name="Joint_4">
-                <command_interface name="position"/>
-                <state_interface name="position">
-                  <param name="initial_value">0.0</param>
-                </state_interface>
-            </joint>
-            <joint name="Joint_5">
-                <command_interface name="position"/>
-                <state_interface name="position">
-                  <param name="initial_value">0.0</param>
-                </state_interface>
-            </joint>
-            <joint name="Joint_6">
-                <command_interface name="position"/>
-                <state_interface name="position">
-                  <param name="initial_value">0.0</param>
-                </state_interface>
-            </joint>
-        </ros2_control>
+  <ros2_control name="Volvo" type="system">
+    <hardware>
+      <plugin>volvo_hardware_interface/VolvoHardwareInterface</plugin>
+      <param name="serial_port">/dev/ttyUSB0</param>
+    </hardware>
+    <joint name="Joint_1">
+        <command_interface name="position"/>
+        <state_interface name="position">
+          <param name="initial_value">0.0</param>
+        </state_interface>
+    </joint>
+    <joint name="Joint_2">
+        <command_interface name="position"/>
+        <state_interface name="position">
+          <param name="initial_value">0.0</param>
+        </state_interface>
+    </joint>
+    <joint name="Joint_3">
+        <command_interface name="position"/>
+        <state_interface name="position">
+          <param name="initial_value">0.0</param>
+        </state_interface>
+    </joint>
+    <joint name="Joint_4">
+        <command_interface name="position"/>
+        <state_interface name="position">
+          <param name="initial_value">0.0</param>
+        </state_interface>
+    </joint>
+    <joint name="Joint_5">
+        <command_interface name="position"/>
+        <state_interface name="position">
+          <param name="initial_value">0.0</param>
+        </state_interface>
+    </joint>
+    <joint name="Joint_6">
+        <command_interface name="position"/>
+        <state_interface name="position">
+          <param name="initial_value">0.0</param>
+        </state_interface>
+    </joint>
+  </ros2_control>
 </robot>
